Commit message: 修复车门位姿 + 新建曲面喷涂轨迹规划器框架
Agent-Logs-Url: https://github.com/username090090009/ros111/sessions/b0821e8e-041c-4318-822c-4922d8d99bac

Co-authored-by: username090090009 <166367875+username090090009@users.noreply.github.com>

File: src/arm_description/urdf/arm_description.xacro (robot description, xacro)
@@ -324,8 +324,21 @@
     <origin xyz="0.05 0 0" rpy="-1.5708 0 -1.5708"/>
   </joint>
+  <!--
+    world_to_door_joint — 车门在世界坐标系中的位姿
+    ================================================
+    xyz: 车门中心到机械臂基座的距离
+      - X = 0.90m：车门中心距机械臂基座 0.9 米（用户设定值）
+      - Y = 0.00m：车门在机械臂正前方
+      - Z = 0.50m：车门中心高度，使喷涂区域处于机械臂可达空间
+    rpy: 车门朝向
+      - yaw = π/2 (1.5708)：将车门旋转 90°，使其平面正对机械臂
+        车门 STL 的厚度方向为 Y 轴，旋转后厚度方向沿世界 X 轴，
+        车门表面法向量指向 -X 方向（朝向机械臂）
+      注：如果加载后车门外表面朝向不对，可将 yaw 改为 -1.5708
+  -->
   <joint name="world_to_door_joint" type="fixed">
     <parent link="world"/>
     <child link="door_link"/>
-    <origin xyz="0.90 0.00 0.00" rpy="0 0 0"/>
+    <origin xyz="0.90 0.00 0.50" rpy="0 0 1.5708"/>
   </joint>
   <!-- Transmissions for ROS Control -->

File: src/arm_description/urdf/door.xacro (robot description, xacro)
@@ -1,4 +1,23 @@
 <?xml version="1.0"?>
+<!--
+  door.xacro — 车门工件模型
+  ==========================
+  车门 STL 由 SolidWorks 导出，坐标单位为毫米（mm），在 URDF 中通过
+  scale="0.001 0.001 0.001" 转换为米。
+  STL 网格包围盒（mm）：
+    X: 1429 ~ 2642  (宽度 ≈ 1213mm)
+    Y: -858 ~ -480  (厚度 ≈ 379mm)
+    Z:  367 ~ 1483  (高度 ≈ 1116mm)
+  网格几何中心（mm）：(2035, -669, 925)
+  对应缩放后（m）：  (2.035, -0.669, 0.925)
+  由于 STL 原点不在网格中心，需要在 visual/collision 的 <origin> 中
+  设置偏移量 xyz="-2.035 0.669 -0.925"，使车门网格居中于 door_link 坐标原点。
+  这样 world_to_door_joint 的 xyz 就直接代表车门中心在世界坐标系中的位置。
+-->
 <robot name="door_panel" xmlns:xacro="http://ros.org/wiki/xacro">
+  <!-- 车门网格几何中心偏移（单位：m），用于将 STL 网格居中到 link 原点 -->
+  <xacro:property name="door_mesh_offset_x" value="-2.035"/>
+  <xacro:property name="door_mesh_offset_y" value="0.669"/>
+  <xacro:property name="door_mesh_offset_z" value="-0.925"/>
   <link name="door_link">
     <inertial>
@@ -9,6 +28,7 @@
                izz="0.2"/>
     </inertial>
+    <!-- 车门可视网格：偏移至 link 原点居中 -->
     <visual>
-      <origin xyz="0 0 0" rpy="0 0 0"/>
+      <origin xyz="${door_mesh_offset_x} ${door_mesh_offset_y} ${door_mesh_offset_z}" rpy="0 0 0"/>
       <geometry>
         <mesh filename="package://arm_description/meshes/car_door_visual.stl" scale="0.001 0.001 0.001"/>
@@ -18,6 +38,7 @@
       </material>
     </visual>
+    <!-- 车门碰撞网格：偏移与 visual 保持一致 -->
     <collision>
-      <origin xyz="0 0 0" rpy="0 0 0"/>
+      <origin xyz="${door_mesh_offset_x} ${door_mesh_offset_y} ${door_mesh_offset_z}" rpy="0 0 0"/>
       <geometry>
         <mesh filename="package://arm_description/meshes/car_door_collision.stl" scale="0.001 0.001 0.001"/>

Commit message: Fix planning timeout: increase IK solver timeout, add IK pre-check, segment-wise execution, diagnostics, collision allowance, orientation relaxation, work frame support, English log messages
Agent-Logs-Url: https://github.com/username090090009/ros111/sessions/e18205ae-e07a-49ce-a1c4-7ce202f08614

Co-authored-by: username090090009 <166367875+username090090009@users.noreply.github.com>

File: src/arm_description/urdf/arm_description.xacro (robot description, xacro)
@@ -341,4 +341,26 @@
     <child link="door_link"/>
     <origin xyz="0.90 0.00 0.50" rpy="0 0 1.5708"/>
+  </joint>
+  <!--
+    door_mount_frame — 车门安装参考坐标系
+    与 door_link 原点重合，用于表示车门的安装位置。
+    在实际部署中，通过标定确定此 frame 在 world 中的位姿。
+  -->
+  <link name="door_mount_frame"/>
+  <joint name="door_to_mount_frame_joint" type="fixed">
+    <parent link="door_link"/>
+    <child link="door_mount_frame"/>
+    <origin xyz="0 0 0" rpy="0 0 0"/>
+  </joint>
+  <!--
+    door_work_frame — 车门喷涂工作坐标系
+    与 door_link 原点重合。喷涂路径点可相对此 frame 表示，
+    便于标定后直接复用路径数据。
+  -->
+  <link name="door_work_frame"/>
+  <joint name="door_to_work_frame_joint" type="fixed">
+    <parent link="door_link"/>
+    <child link="door_work_frame"/>
+    <origin xyz="0 0 0" rpy="0 0 0"/>
   </joint>
   <!-- Transmissions for ROS Control -->
